Commit message: added tags to mannequin by changing directory

File: aruco_tags/src/arucobaxter_gazebo/urdf/09-publishjoints.urdf.xacro (robot description, xacro)
@@ -114,5 +114,5 @@
       <origin rpy="0 ${pi/2} 0" xyz="0.1 0 -0.5"/>
       <geometry>
-        <mesh filename="package://urdf_tutorial/meshes/arucotag1.dae"/>
+        <mesh filename="package://arucobaxter_gazebo/meshes/arucotag1.dae"/>
       </geometry>
     </visual>
@@ -126,5 +126,5 @@
       <origin rpy="0 ${pi/2} 0" xyz="0.1 0 -0.1"/>
       <geometry>
-        <mesh filename="package://urdf_tutorial/meshes/arucotag1.dae"/>
+        <mesh filename="package://arucobaxter_gazebo/meshes/arucotag1.dae"/>
       </geometry>
     </visual>
