Commit message: adding manual movements

File: final_ws/src/aruco_planning/urdf/09-publishjoints.urdf.xacro (robot description, xacro)
@@ -43,4 +43,8 @@
   <xacro:macro name="arm" params="prefix reflect">
     <link name="${prefix}_arm">
+      <!-- <inertial>
+          <mass value="0.18" />
+          <inertia ixx="0.5" ixy="0.0" ixz="0.0" iyy="0.5" iyz="0.0" izz="0.5" />
+      </inertial> -->
       <visual>
         <geometry>

Commit message: controlled humanbot

File: final_ws/src/aruco_planning/urdf/09-publishjoints.urdf.xacro (robot description, xacro)
@@ -17,7 +17,4 @@
     <color rgba="1 1 1 1"/>
   </material>
-  <gazebo reference="base_link">
-   <turnGravityOn>true</turnGravityOn>
-  </gazebo>
   <xacro:macro name="default_inertial" params="mass">
     <inertial>
@@ -43,8 +40,9 @@
   <xacro:macro name="arm" params="prefix reflect">
     <link name="${prefix}_arm">
-      <!-- <inertial>
-          <mass value="0.18" />
-          <inertia ixx="0.5" ixy="0.0" ixz="0.0" iyy="0.5" iyz="0.0" izz="0.5" />
-      </inertial> -->
+      <inertial>
+        <origin rpy="0 0 0" xyz="0 0 0"/>
+        <mass value="10"/>
+        <inertia ixx="0.308" ixy="0.0" ixz="0.0" iyy="0.04" iyz="0.0" izz="0.333"/>
+      </inertial>
       <visual>
         <geometry>
@@ -60,12 +58,12 @@
         <origin xyz="0 0 -${leglen}" rpy="0 ${pi/2} 0"/>
       </collision>
-      <xacro:default_inertial mass="10"/>
     </link>
     <joint name="base_to_${prefix}_arm" type="revolute">
       <axis xyz="1 0 0"/>
-      <limit effort="50.0" lower="0.0" upper="${reflect *3}" velocity="1"/>
+      <limit effort="50000.0" lower="0.0" upper="${reflect *3}" velocity="0.000001"/>
       <origin rpy="0 0 0" xyz="0 ${reflect*(width+.02)} 0.85" />
       <parent link="base_link"/>
       <child link="${prefix}_arm"/>
+      <dynamics damping="0.05" friction="0"/>
     </joint>
   </xacro:macro>
@@ -121,5 +119,5 @@
       <origin rpy="0 ${pi/2} 0" xyz="0.1 0 -0.5"/>
       <geometry>
-        <mesh filename="package://aruco_planning/meshes/arucotag1.dae"/>
+        <mesh filename="package://urdf_tutorial/meshes/arucotag1.dae"/>
       </geometry>
     </visual>
@@ -133,5 +131,5 @@
       <origin rpy="0 ${pi/2} 0" xyz="0.1 0 -0.1"/>
       <geometry>
-        <mesh filename="package://aruco_planning/meshes/arucotag1.dae"/>
+        <mesh filename="package://urdf_tutorial/meshes/arucotag1.dae"/>
       </geometry>
     </visual>
@@ -147,3 +145,11 @@
     </plugin>
   </gazebo>
+    <gazebo reference="base_link">
+    <mu1>0</mu1>
+    <mu2>0</mu2>
+    <fdir1 value = "1 0 0"/>
+ <dynamics damping="0.7" friction="100.0" />
+    <material>Gazebo/Black</material>
+    <turnGravityOff>false</turnGravityOff>
+  </gazebo>
 </robot>

Commit message: pedistal humanbot

File: final_ws/src/aruco_planning/urdf/09-publishjoints.urdf.xacro (robot description, xacro)
@@ -8,4 +8,5 @@
   <xacro:property name="wheeldiam" value="0.07" />
   <xacro:property name="pi" value="3.1415" />
+  <xacro:property name="ped_height" value="0.8" />
   <material name="blue">
     <color rgba="0 0 0.8 1"/>
@@ -28,5 +29,5 @@
         <cylinder radius="${width}" length="${bodylen}"/>
       </geometry>
-      <origin xyz="0 0 0.6"/>
+      <origin xyz="0 0 ${0.6+ped_height}"/>
       <material name="blue"/>
     </visual>
@@ -56,5 +57,5 @@
           <box size="${leglen/2} 0.1 0.2"/>
         </geometry>
-        <origin xyz="0 0 -${leglen}" rpy="0 ${pi/2} 0"/>
+        <origin xyz="0 0 -${leglen+ped_height}" rpy="0 ${pi/2} 0"/>
       </collision>
     </link>
@@ -62,8 +63,8 @@
       <axis xyz="1 0 0"/>
       <limit effort="50000.0" lower="0.0" upper="${reflect *3}" velocity="0.000001"/>
-      <origin rpy="0 0 0" xyz="0 ${reflect*(width+.02)} 0.85" />
+      <origin rpy="0 0 0" xyz="0 ${reflect*(width+.02)} ${0.85+ped_height}" />
       <parent link="base_link"/>
       <child link="${prefix}_arm"/>
-      <dynamics damping="0.05" friction="0"/>
+      <dynamics damping="0.1" friction="0"/>
     </joint>
   </xacro:macro>
@@ -90,5 +91,5 @@
       <parent link="base_link"/>
       <child link="${prefix}_leg"/>
-      <origin xyz="0 ${reflect*0.1} 0.25" />
+      <origin xyz="0 ${reflect*0.1} ${0.25+ped_height}" />
     </joint>
   </xacro:macro>
@@ -113,9 +114,9 @@
     <child link="head"/>
     <axis xyz="0 0 1"/>
-    <origin xyz="0 0 1.1"/>
+    <origin xyz="0 0 ${1.1+ped_height}"/>
   </joint>
   <link name="aruco1">
     <visual>
-      <origin rpy="0 ${pi/2} 0" xyz="0.1 0 -0.5"/>
+      <origin rpy="0 ${pi/2} 0" xyz="0.1 0 ${-0.5}"/>
       <geometry>
         <mesh filename="package://urdf_tutorial/meshes/arucotag1.dae"/>
@@ -127,5 +128,26 @@
     <child link="aruco1"/>
   </joint>
-   <link name="aruco2">
+    <link name="pedistal">
+      <visual>
+        <geometry>
+          <box size="0.8 0.8 0.8"/>
+        </geometry>
+        <origin xyz="0 0 0" rpy="0 ${pi/2} 0"/>
+        <material name="black"/>
+      </visual>
+      <collision>
+        <geometry>
+          <box size="0.5 0.5 ${ped_height}"/>
+        </geometry>
+        <origin xyz="0 0 0" rpy="0 ${pi/2} 0"/>
+      </collision>
+      <xacro:default_inertial mass="10"/>
+    </link>
+    <joint name="leg_pedistal" type="fixed">
+      <parent link="base_link"/>
+      <child link="pedistal"/>
+      <origin xyz="0 0 0" />
+    </joint>
+<!--    <link name="aruco2">
     <visual>
       <origin rpy="0 ${pi/2} 0" xyz="0.1 0 -0.1"/>
@@ -139,4 +161,5 @@
     <child link="aruco2"/>
   </joint>
+ -->
   <!-- Gazebo plugin for ROS Control -->
   <gazebo>

Commit message: adding new pedistal box file

File: final_ws/src/aruco_planning/urdf/09-publishjoints.urdf.xacro (robot description, xacro)
@@ -8,5 +8,4 @@
   <xacro:property name="wheeldiam" value="0.07" />
   <xacro:property name="pi" value="3.1415" />
-  <xacro:property name="ped_height" value="0.8" />
   <material name="blue">
     <color rgba="0 0 0.8 1"/>
@@ -29,5 +28,5 @@
         <cylinder radius="${width}" length="${bodylen}"/>
       </geometry>
-      <origin xyz="0 0 ${0.6+ped_height}"/>
+      <origin xyz="0 0 0.6"/>
       <material name="blue"/>
     </visual>
@@ -57,5 +56,5 @@
           <box size="${leglen/2} 0.1 0.2"/>
         </geometry>
-        <origin xyz="0 0 -${leglen+ped_height}" rpy="0 ${pi/2} 0"/>
+        <origin xyz="0 0 -${leglen}" rpy="0 ${pi/2} 0"/>
       </collision>
     </link>
@@ -63,8 +62,8 @@
       <axis xyz="1 0 0"/>
       <limit effort="50000.0" lower="0.0" upper="${reflect *3}" velocity="0.000001"/>
-      <origin rpy="0 0 0" xyz="0 ${reflect*(width+.02)} ${0.85+ped_height}" />
+      <origin rpy="0 0 0" xyz="0 ${reflect*(width+.02)} 0.85" />
       <parent link="base_link"/>
       <child link="${prefix}_arm"/>
-      <dynamics damping="0.1" friction="0"/>
+      <dynamics damping="0.05" friction="0"/>
     </joint>
   </xacro:macro>
@@ -91,5 +90,5 @@
       <parent link="base_link"/>
       <child link="${prefix}_leg"/>
-      <origin xyz="0 ${reflect*0.1} ${0.25+ped_height}" />
+      <origin xyz="0 ${reflect*0.1} 0.25" />
     </joint>
   </xacro:macro>
@@ -114,9 +113,9 @@
     <child link="head"/>
     <axis xyz="0 0 1"/>
-    <origin xyz="0 0 ${1.1+ped_height}"/>
+    <origin xyz="0 0 1.1"/>
   </joint>
   <link name="aruco1">
     <visual>
-      <origin rpy="0 ${pi/2} 0" xyz="0.1 0 ${-0.5}"/>
+      <origin rpy="0 ${pi/2} 0" xyz="0.1 0 -0.5"/>
       <geometry>
         <mesh filename="package://urdf_tutorial/meshes/arucotag1.dae"/>
@@ -128,26 +127,6 @@
     <child link="aruco1"/>
   </joint>
-    <link name="pedistal">
-      <visual>
-        <geometry>
-          <box size="0.8 0.8 0.8"/>
-        </geometry>
-        <origin xyz="0 0 0" rpy="0 ${pi/2} 0"/>
-        <material name="black"/>
-      </visual>
-      <collision>
-        <geometry>
-          <box size="0.5 0.5 ${ped_height}"/>
-        </geometry>
-        <origin xyz="0 0 0" rpy="0 ${pi/2} 0"/>
-      </collision>
-      <xacro:default_inertial mass="10"/>
-    </link>
-    <joint name="leg_pedistal" type="fixed">
-      <parent link="base_link"/>
-      <child link="pedistal"/>
-      <origin xyz="0 0 0" />
-    </joint>
-<!--    <link name="aruco2">
+<!--
+   <link name="aruco2">
     <visual>
       <origin rpy="0 ${pi/2} 0" xyz="0.1 0 -0.1"/>
@@ -160,6 +139,5 @@
     <parent link="left_arm"/>
     <child link="aruco2"/>
-  </joint>
- -->
+  </joint> -->
   <!-- Gazebo plugin for ROS Control -->
   <gazebo>
